Commit message: Fix simulation to follow the path

File: path2d/joint_robot.urdf (robot description, URDF)
Before this commit: robot mmp_panda, 6 links, 5 joints
Links:
- link linkTool: geometry visual box size=0.08 0.02 0.01; visual cylinder length=0.1 radius=0.01
Joints:
- joint jointTool: type prismatic -> fixed
